Commit message: Add real and sim robot toggle functionality

File: lidarbot_description/urdf/lidarbot.urdf.xacro (robot description, xacro)
@@ -2,4 +2,5 @@
 <robot name="lidarbot" xmlns:xacro="http://ros.org/wiki/xacro">
     <xacro:arg name="use_ros2_control" default="true"/>
+    <xacro:arg name="sim_mode" default="false"/>
     <xacro:include filename="lidarbot_core.xacro"/>
     <xacro:if value="$(arg use_ros2_control)">

File: lidarbot_description/urdf/ros2_control.xacro (robot description, xacro)
@@ -1,52 +1,59 @@
 <?xml version="1.0" ?>
 <robot xmlns:xacro="http://ros.org/wiki/xacro">
-  <ros2_control name='RealRobot' type='system'>
-    <hardware>
-      <plugin>lidarbot_base/LidarbotHardware</plugin>
-        <param name="left_wheel_name">left_wheel_joint</param>
-        <param name="right_wheel_name">right_wheel_joint</param>
-        <param name="enc_ticks_per_rev">20</param>
-    </hardware>
-    <joint name='left_wheel_joint'>
-      <command_interface name='velocity'>
-        <param name='min'>-10</param>
-        <param name='max'>10</param>
-      </command_interface>
-      <state_interface name='velocity'/>
-      <state_interface name='position'/>
-    </joint>
-    <joint name='right_wheel_joint'>
-      <command_interface name='velocity'>
-        <param name='min'>-10</param>
-        <param name='max'>10</param>
-      </command_interface>
-      <state_interface name='velocity'/>
-      <state_interface name='position'/>
-    </joint>
-  </ros2_control>
-  <!-- <ros2_control name='GazeboSystem' type='system'>
-    <hardware>
-      <plugin>gazebo_ros2_control/GazeboSystem</plugin>
-    </hardware>
-    <joint name='left_wheel_joint'>
-      <command_interface name='velocity'>
-        <param name='min'>-10</param>
-        <param name='max'>10</param>
-      </command_interface>
-      <state_interface name='velocity'/>
-      <state_interface name='position'/>
-    </joint>
-    <joint name='right_wheel_joint'>
-      <command_interface name='velocity'>
-        <param name='min'>-10</param>
-        <param name='max'>10</param>
-      </command_interface>
-      <state_interface name='velocity'/>
-      <state_interface name='position'/>
-    </joint>
-  </ros2_control> -->
+  <!-- Real robot ros2_control -->
+  <xacro:unless value="$(arg sim_mode)">
+    <ros2_control name='RealRobot' type='system'>
+      <hardware>
+        <plugin>lidarbot_base/LidarbotHardware</plugin>
+          <param name="left_wheel_name">left_wheel_joint</param>
+          <param name="right_wheel_name">right_wheel_joint</param>
+          <param name="enc_ticks_per_rev">20</param>
+      </hardware>
+      <joint name='left_wheel_joint'>
+        <command_interface name='velocity'>
+          <param name='min'>-10</param>
+          <param name='max'>10</param>
+        </command_interface>
+        <state_interface name='velocity'/>
+        <state_interface name='position'/>
+      </joint>
+      <joint name='right_wheel_joint'>
+        <command_interface name='velocity'>
+          <param name='min'>-10</param>
+          <param name='max'>10</param>
+        </command_interface>
+        <state_interface name='velocity'/>
+        <state_interface name='position'/>
+      </joint>
+    </ros2_control>
+  </xacro:unless>
+  <!-- Gazebo ros2_control -->
+  <xacro:if value="$(arg sim_mode)">
+    <ros2_control name='GazeboSystem' type='system'>
+      <hardware>
+        <plugin>gazebo_ros2_control/GazeboSystem</plugin>
+      </hardware>
+      <joint name='left_wheel_joint'>
+        <command_interface name='velocity'>
+          <param name='min'>-10</param>
+          <param name='max'>10</param>
+        </command_interface>
+        <state_interface name='velocity'/>
+        <state_interface name='position'/>
+      </joint>
+      <joint name='right_wheel_joint'>
+        <command_interface name='velocity'>
+          <param name='min'>-10</param>
+          <param name='max'>10</param>
+        </command_interface>
+        <state_interface name='velocity'/>
+        <state_interface name='position'/>
+      </joint>
+    </ros2_control>
+  </xacro:if>
   <gazebo>
     <plugin name='gazebo_ros2_control' filename='libgazebo_ros2_control.so'>
       <parameters>$(find lidarbot_bringup)/config/controllers.yaml</parameters>
+      <parameters>$(find lidarbot_bringup)/config/gazebo_ros2_ctl_use_sim.yaml</parameters>
     </plugin>
   </gazebo>
