Commit message: Fix lidar to display in rviz

File: lidarbot_description/urdf/lidar.xacro (robot description, xacro)
@@ -13,47 +13,47 @@
             </geometry>
         </collision>
-        </link>
-        <joint name="lidar_joint" type="fixed">
-            <parent link="chassis_link"/>
-            <child link="lidar_link"/>
-            <origin xyz="0.0335 0.0095 0.069" rpy="0 0 0"/>
-            <axis xyz="0 0 1"/>
-        </joint>
-        <xacro:cylinder_inertia mass="${wheel_mass}" length="0.021" radius="0.037">
+         <xacro:cylinder_inertia mass="${wheel_mass}" length="0.021" radius="0.037">
             <origin xyz="0 0 0" rpy="0 0 0"/>
         </xacro:cylinder_inertia>
-        <gazebo reference="lidar_link">
-            <sensor name="lidar" type="ray">
-                <pose> 0 0 0 0 0 0 </pose>
-                <visualize>false</visualize>
-                <update_rate>5.5</update_rate>
-                <ray>
-                    <scan>
-                        <horizontal>
-                            <samples>360</samples>
-                            <resolution>1</resolution>
-                            <min_angle>-3.14</min_angle>
-                            <max_angle>3.14</max_angle>
-                        </horizontal>
-                    </scan>
-                    <range>
-                        <min>0.15</min>
-                        <max>12</max>
-                        <resolution>0.2</resolution>
-                    <noise>
-                        <type>gaussian</type>
-                        <mean>0.0</mean>
-                        <stddev>0.01</stddev>
-                    </noise>
-                    </range>
-                </ray>
-                <plugin name="lidar_controller" filename="libgazebo_ros_ray_sensor.so">
-                    <ros>
-                        <remapping>~/out:=scan</remapping>
-                    </ros>
-                    <output_type>sensor_msgs/LaserScan</output_type>
-                    <frame_name>lidar_link</frame_name>
-                </plugin>
-            </sensor>
-        </gazebo>
+   </link>
+    <joint name="lidar_joint" type="fixed">
+        <parent link="chassis_link"/>
+        <child link="lidar_link"/>
+        <origin xyz="0.0335 0.0095 0.069" rpy="0 0 ${-pi/2}"/>
+        <axis xyz="0 0 1"/>
+    </joint>
+    <gazebo reference="lidar_link">
+        <sensor name="lidar" type="ray">
+            <pose> 0 0 0 0 0 0 </pose>
+            <visualize>false</visualize>
+            <update_rate>5.5</update_rate>
+            <ray>
+                <scan>
+                    <horizontal>
+                        <samples>360</samples>
+                        <resolution>1</resolution>
+                        <min_angle>-3.14</min_angle>
+                        <max_angle>3.14</max_angle>
+                    </horizontal>
+                </scan>
+                <range>
+                    <min>0.15</min>
+                    <max>12</max>
+                    <resolution>0.2</resolution>
+                <noise>
+                    <type>gaussian</type>
+                    <mean>0.0</mean>
+                    <stddev>0.01</stddev>
+                </noise>
+                </range>
+            </ray>
+            <plugin name="lidar_controller" filename="libgazebo_ros_ray_sensor.so">
+                <ros>
+                    <remapping>~/out:=scan</remapping>
+                </ros>
+                <output_type>sensor_msgs/LaserScan</output_type>
+                <frame_name>lidar_link</frame_name>
+            </plugin>
+        </sensor>
+    </gazebo>
 </robot>
