Commit message: Update xacro files to fix rviz frame issue

File: lidarbot_description/urdf/camera.xacro (robot description, xacro)
@@ -17,5 +17,5 @@
   </link>
   <joint name="camera_joint" type="fixed">
-    <parent link="base_link"/>
+    <parent link="chassis_link"/>
     <child link="camera_link"/>
     <origin xyz="0.1 0 0.0425" rpy="0 0 0"/>

File: lidarbot_description/urdf/gazebo_control.xacro (robot description, xacro)
@@ -13,5 +13,5 @@
             <!-- Output -->
             <odometry_frame>odom</odometry_frame>
-            <robot_base_frame>base_footprint</robot_base_frame>
+            <robot_base_frame>base_link</robot_base_frame>
             <publish_odom>true</publish_odom>
             <publish_odom_tf>true</publish_odom_tf>

File: lidarbot_description/urdf/imu.xacro (robot description, xacro)
@@ -10,5 +10,5 @@
   </link>
   <joint name="imu_joint" type="fixed">
-    <parent link="base_link"/>
+    <parent link="chassis_link"/>
     <child link="imu_link"/>
     <origin xyz="-0.06 0 0.0175" rpy="0 0 ${pi}"/>

File: lidarbot_description/urdf/lidar.xacro (robot description, xacro)
@@ -15,5 +15,5 @@
         </link>
         <joint name="lidar_joint" type="fixed">
-            <parent link="base_link"/>
+            <parent link="chassis_link"/>
             <child link="lidar_link"/>
             <origin xyz="0.0335 0.0095 0.069" rpy="0 0 0"/>

File: lidarbot_description/urdf/lidarbot_core.xacro (robot description, xacro)
@@ -12,17 +12,17 @@
   <!-- Distance between centre of wheel and robot base/chassis -->
   <xacro:property name="wheel_zoff" value="0.0125"/>
-  <!-- Robot Base Footprint - the centre of the main robot chassis projected on the ground -->
-  <link name="base_footprint"/>
-  <joint name="base_joint" type="fixed">
-    <parent link="base_footprint"/>
-    <child link="base_link"/>
-    <origin xyz="0 0 ${(wheel_radius+wheel_zoff)}" rpy="0 0 0"/>
-  </joint>
-  <!-- Robot Base -->
-  <link name="base_link">
+   <!-- Base link -->
+   <link name="base_link"/>
+   <joint name="chassis_joint" type="fixed">
+     <parent link="base_link"/>
+     <child link="chassis_link"/>
+     <origin xyz="0 0 -${(wheel_radius+wheel_zoff)}" rpy="0 0 0"/>
+   </joint>
+  <!-- Robot Chassis -->
+  <link name="chassis_link">
       <visual>
         <origin xyz="0 0 ${-wheel_zoff}" rpy="0 0 0"/>
           <geometry>
-              <mesh filename="file://$(find lidarbot_description)/meshes/robot_base.dae" />
+              <mesh filename="file://$(find lidarbot_description)/meshes/robot_chassis.dae" />
           </geometry>
       </visual>
@@ -158,5 +158,5 @@
   </link>
   <joint name="left_wheel_joint" type="continuous">
-    <parent link="base_link"/>
+    <parent link="chassis_link"/>
     <child link="left_wheel"/>
     <origin xyz="-0.028 0.055 -${wheel_zoff}" rpy="${pi/2} 0 ${pi}"/>
@@ -181,5 +181,5 @@
   </link>
   <joint name="right_wheel_joint" type="continuous">
-    <parent link="base_link"/>
+    <parent link="chassis_link"/>
     <child link="right_wheel"/>
     <origin xyz="-0.028 -0.065 -${wheel_zoff}" rpy="${pi/2} 0 ${-pi}"/>
@@ -204,5 +204,5 @@
   </link>
   <joint name="caster_wheel_joint" type="fixed">
-    <parent link="base_link"/>
+    <parent link="chassis_link"/>
     <child link="caster_wheel"/>
     <origin xyz="0.0925 0 -0.031" rpy="0 0 ${pi/2}"/>

Commit message: Refactor packages for rviz mesh file compatibility

File: lidarbot_description/urdf/camera.xacro (robot description, xacro)
@@ -6,5 +6,5 @@
       <origin xyz="0 0 0" rpy="${pi/2} 0 ${pi/2}"/>
       <geometry>
-        <mesh filename="file://$(find lidarbot_description)/meshes/d415.dae"/>
+        <mesh filename="package://lidarbot_description/meshes/d415.dae"/>
       </geometry>
     </visual>

File: lidarbot_description/urdf/imu.xacro (robot description, xacro)
@@ -5,5 +5,5 @@
     <visual name="imu_visual">
       <geometry>
-        <mesh filename="file://$(find lidarbot_description)/meshes/MPU6050.dae"/>
+        <mesh filename="package://lidarbot_description/meshes/MPU6050.dae"/>
       </geometry>
     </visual>

File: lidarbot_description/urdf/lidar.xacro (robot description, xacro)
@@ -4,5 +4,5 @@
         <visual>
             <geometry>
-            <mesh filename="file://$(find lidarbot_description)/meshes/rplidar_top.dae"/>
+            <mesh filename="package://lidarbot_description/meshes/rplidar_top.dae"/>
             </geometry>
         </visual>

File: lidarbot_description/urdf/lidarbot_core.xacro (robot description, xacro)
@@ -24,5 +24,5 @@
         <origin xyz="0 0 ${-wheel_zoff}" rpy="0 0 0"/>
           <geometry>
-              <mesh filename="file://$(find lidarbot_description)/meshes/robot_chassis.dae" />
+              <mesh filename="package://lidarbot_description/meshes/robot_chassis.dae" />
           </geometry>
       </visual>
@@ -36,5 +36,5 @@
           <origin xyz="0.086 0 -0.0475" rpy="0 0 0"/>
         <geometry>
-          <mesh filename="file://$(find lidarbot_description)/meshes/caster_mount.dae" />
+          <mesh filename="package://lidarbot_description/meshes/caster_mount.dae" />
         </geometry>
       </visual>
@@ -49,5 +49,5 @@
         <origin xyz="-0.06 0.015 0.031" rpy="${pi} 0 ${-pi}"/>
           <geometry>
-              <mesh filename="file://$(find lidarbot_description)/meshes/rpi_stand.dae" />
+              <mesh filename="package://lidarbot_description/meshes/rpi_stand.dae" />
           </geometry>
       </visual>
@@ -62,5 +62,5 @@
         <origin xyz="-0.059 0.00245 0.033" rpy="0 0 ${pi/2}"/>
         <geometry>
-          <mesh filename="file://$(find lidarbot_description)/meshes/rpi_4.dae"/>
+          <mesh filename="package://lidarbot_description/meshes/rpi_4.dae"/>
         </geometry>
       </visual>
@@ -75,5 +75,5 @@
         <origin xyz="0.033 0.015 0.031" rpy="${pi} 0 ${pi}"/>
         <geometry>
-          <mesh filename="file://$(find lidarbot_description)/meshes/power_bank_stand.dae"/>
+          <mesh filename="package://lidarbot_description/meshes/power_bank_stand.dae"/>
         </geometry>
       </visual>
@@ -88,5 +88,5 @@
         <origin xyz="0.0635 0.04775 0.015" rpy="0 0 ${pi/2}"/>
         <geometry>
-          <mesh filename="file://$(find lidarbot_description)/meshes/power_bank.dae"/>
+          <mesh filename="package://lidarbot_description/meshes/power_bank.dae"/>
         </geometry>
       </visual>
@@ -101,5 +101,5 @@
         <origin xyz="0.033 0.015 0.017" rpy="0 0 ${-2*pi}"/>
         <geometry>
-          <mesh filename="file://$(find lidarbot_description)/meshes/rplidar_stand.dae"/>
+          <mesh filename="package://lidarbot_description/meshes/rplidar_stand.dae"/>
         </geometry>
       </visual>
@@ -114,5 +114,5 @@
         <origin xyz="0.03485 0.0087 0.037" rpy="0 0 ${-pi/2}"/>
           <geometry>
-            <mesh filename="file://$(find lidarbot_description)/meshes/rplidar_base.dae"/>
+            <mesh filename="package://lidarbot_description/meshes/rplidar_base.dae"/>
           </geometry>
         </visual>
@@ -144,5 +144,5 @@
     <visual>
         <geometry>
-          <mesh filename="file://$(find lidarbot_description)/meshes/left_wheel.dae" />
+          <mesh filename="package://lidarbot_description/meshes/left_wheel.dae" />
         </geometry>
     </visual>
@@ -167,5 +167,5 @@
     <visual>
       <geometry>
-        <mesh filename="file://$(find lidarbot_description)/meshes/right_wheel.dae"/>
+        <mesh filename="package://lidarbot_description/meshes/right_wheel.dae"/>
       </geometry>
     </visual>
@@ -190,5 +190,5 @@
     <visual>
       <geometry>
-        <mesh filename="file://$(find lidarbot_description)/meshes/caster_wheel.dae"/>
+        <mesh filename="package://lidarbot_description/meshes/caster_wheel.dae"/>
       </geometry>
     </visual>

Commit message: Revert to previous mesh file include format

File: lidarbot_description/urdf/camera.xacro (robot description, xacro)
@@ -6,5 +6,6 @@
       <origin xyz="0 0 0" rpy="${pi/2} 0 ${pi/2}"/>
       <geometry>
-        <mesh filename="package://lidarbot_description/meshes/d415.dae"/>
+        <mesh filename="file://$(find lidarbot_description)/meshes/d415.dae"/>
+        <!-- <mesh filename="package://lidarbot_description/meshes/d415.dae"/> -->
       </geometry>
     </visual>

File: lidarbot_description/urdf/imu.xacro (robot description, xacro)
@@ -5,5 +5,6 @@
     <visual name="imu_visual">
       <geometry>
-        <mesh filename="package://lidarbot_description/meshes/MPU6050.dae"/>
+        <mesh filename="file://$(find lidarbot_description)/meshes/MPU6050.dae"/>
+        <!-- <mesh filename="package://lidarbot_description/meshes/MPU6050.dae"/> -->
       </geometry>
     </visual>

File: lidarbot_description/urdf/lidar.xacro (robot description, xacro)
@@ -4,5 +4,6 @@
         <visual>
             <geometry>
-            <mesh filename="package://lidarbot_description/meshes/rplidar_top.dae"/>
+            <mesh filename="file://$(find lidarbot_description)/meshes/rplidar_top.dae"/>
+            <!-- <mesh filename="package://lidarbot_description/meshes/rplidar_top.dae"/> -->
             </geometry>
         </visual>

File: lidarbot_description/urdf/lidarbot_core.xacro (robot description, xacro)
@@ -24,5 +24,6 @@
         <origin xyz="0 0 ${-wheel_zoff}" rpy="0 0 0"/>
           <geometry>
-              <mesh filename="package://lidarbot_description/meshes/robot_chassis.dae" />
+              <mesh filename="file://$(find lidarbot_description)/meshes/robot_chassis.dae" />
+              <!-- <mesh filename="package://lidarbot_description/meshes/robot_chassis.dae" /> -->
           </geometry>
       </visual>
@@ -36,5 +37,6 @@
           <origin xyz="0.086 0 -0.0475" rpy="0 0 0"/>
         <geometry>
-          <mesh filename="package://lidarbot_description/meshes/caster_mount.dae" />
+          <mesh filename="file://$(find lidarbot_description)/meshes/caster_mount.dae" />
+          <!-- <mesh filename="package://lidarbot_description/meshes/caster_mount.dae" /> -->
         </geometry>
       </visual>
@@ -49,5 +51,6 @@
         <origin xyz="-0.06 0.015 0.031" rpy="${pi} 0 ${-pi}"/>
           <geometry>
-              <mesh filename="package://lidarbot_description/meshes/rpi_stand.dae" />
+              <mesh filename="file://$(find lidarbot_description)/meshes/rpi_stand.dae" />
+              <!-- <mesh filename="package://lidarbot_description/meshes/rpi_stand.dae" /> -->
           </geometry>
       </visual>
@@ -62,5 +65,6 @@
         <origin xyz="-0.059 0.00245 0.033" rpy="0 0 ${pi/2}"/>
         <geometry>
-          <mesh filename="package://lidarbot_description/meshes/rpi_4.dae"/>
+          <mesh filename="file://$(find lidarbot_description)/meshes/rpi_4.dae"/>
+          <!-- <mesh filename="package://lidarbot_description/meshes/rpi_4.dae"/> -->
         </geometry>
       </visual>
@@ -75,5 +79,6 @@
         <origin xyz="0.033 0.015 0.031" rpy="${pi} 0 ${pi}"/>
         <geometry>
-          <mesh filename="package://lidarbot_description/meshes/power_bank_stand.dae"/>
+          <mesh filename="file://$(find lidarbot_description)/meshes/power_bank_stand.dae"/>
+          <!-- <mesh filename="package://lidarbot_description/meshes/power_bank_stand.dae"/> -->
         </geometry>
       </visual>
@@ -88,5 +93,6 @@
         <origin xyz="0.0635 0.04775 0.015" rpy="0 0 ${pi/2}"/>
         <geometry>
-          <mesh filename="package://lidarbot_description/meshes/power_bank.dae"/>
+          <mesh filename="file://$(find lidarbot_description)/meshes/power_bank.dae"/>
+          <!-- <mesh filename="package://lidarbot_description/meshes/power_bank.dae"/> -->
         </geometry>
       </visual>
@@ -101,5 +107,6 @@
         <origin xyz="0.033 0.015 0.017" rpy="0 0 ${-2*pi}"/>
         <geometry>
-          <mesh filename="package://lidarbot_description/meshes/rplidar_stand.dae"/>
+          <mesh filename="file://$(find lidarbot_description)/meshes/rplidar_stand.dae"/>
+          <!-- <mesh filename="package://lidarbot_description/meshes/rplidar_stand.dae"/> -->
         </geometry>
       </visual>
@@ -114,5 +121,6 @@
         <origin xyz="0.03485 0.0087 0.037" rpy="0 0 ${-pi/2}"/>
           <geometry>
-            <mesh filename="package://lidarbot_description/meshes/rplidar_base.dae"/>
+            <mesh filename="file://$(find lidarbot_description)/meshes/rplidar_base.dae"/>
+            <!-- <mesh filename="package://lidarbot_description/meshes/rplidar_base.dae"/> -->
           </geometry>
         </visual>
@@ -144,5 +152,6 @@
     <visual>
         <geometry>
-          <mesh filename="package://lidarbot_description/meshes/left_wheel.dae" />
+          <mesh filename="file://$(find lidarbot_description)/meshes/left_wheel.dae" />
+          <!-- <mesh filename="package://lidarbot_description/meshes/left_wheel.dae" /> -->
         </geometry>
     </visual>
@@ -167,5 +176,6 @@
     <visual>
       <geometry>
-        <mesh filename="package://lidarbot_description/meshes/right_wheel.dae"/>
+        <mesh filename="file://$(find lidarbot_description)/meshes/right_wheel.dae"/>
+        <!-- <mesh filename="package://lidarbot_description/meshes/right_wheel.dae"/> -->
       </geometry>
     </visual>
@@ -190,5 +200,6 @@
     <visual>
       <geometry>
-        <mesh filename="package://lidarbot_description/meshes/caster_wheel.dae"/>
+        <mesh filename="file://$(find lidarbot_description)/meshes/caster_wheel.dae"/>
+        <!-- <mesh filename="package://lidarbot_description/meshes/caster_wheel.dae"/> -->
       </geometry>
     </visual>

Commit message: Minor changes to xacro files

File: lidarbot_description/urdf/camera.xacro (robot description, xacro)
@@ -6,6 +6,6 @@
       <origin xyz="0 0 0" rpy="${pi/2} 0 ${pi/2}"/>
       <geometry>
-        <mesh filename="file://$(find lidarbot_description)/meshes/d415.dae"/>
-        <!-- <mesh filename="package://lidarbot_description/meshes/d415.dae"/> -->
+        <!-- <mesh filename="file://$(find lidarbot_description)/meshes/d415.dae"/> -->
+        <mesh filename="package://lidarbot_description/meshes/d415.dae"/>
       </geometry>
     </visual>

File: lidarbot_description/urdf/imu.xacro (robot description, xacro)
@@ -5,6 +5,6 @@
     <visual name="imu_visual">
       <geometry>
-        <mesh filename="file://$(find lidarbot_description)/meshes/MPU6050.dae"/>
-        <!-- <mesh filename="package://lidarbot_description/meshes/MPU6050.dae"/> -->
+        <!-- <mesh filename="file://$(find lidarbot_description)/meshes/MPU6050.dae"/> -->
+        <mesh filename="package://lidarbot_description/meshes/MPU6050.dae"/>
       </geometry>
     </visual>

File: lidarbot_description/urdf/lidar.xacro (robot description, xacro)
@@ -4,6 +4,6 @@
         <visual>
             <geometry>
-            <mesh filename="file://$(find lidarbot_description)/meshes/rplidar_top.dae"/>
-            <!-- <mesh filename="package://lidarbot_description/meshes/rplidar_top.dae"/> -->
+            <!-- <mesh filename="file://$(find lidarbot_description)/meshes/rplidar_top.dae"/> -->
+            <mesh filename="package://lidarbot_description/meshes/rplidar_top.dae"/>
             </geometry>
         </visual>

File: lidarbot_description/urdf/lidarbot_core.xacro (robot description, xacro)
@@ -24,6 +24,6 @@
         <origin xyz="0 0 ${-wheel_zoff}" rpy="0 0 0"/>
           <geometry>
-              <mesh filename="file://$(find lidarbot_description)/meshes/robot_chassis.dae" />
-              <!-- <mesh filename="package://lidarbot_description/meshes/robot_chassis.dae" /> -->
+              <!-- <mesh filename="file://$(find lidarbot_description)/meshes/robot_chassis.dae" /> -->
+              <mesh filename="package://lidarbot_description/meshes/robot_chassis.dae" />
           </geometry>
       </visual>
@@ -37,6 +37,6 @@
           <origin xyz="0.086 0 -0.0475" rpy="0 0 0"/>
         <geometry>
-          <mesh filename="file://$(find lidarbot_description)/meshes/caster_mount.dae" />
-          <!-- <mesh filename="package://lidarbot_description/meshes/caster_mount.dae" /> -->
+          <!-- <mesh filename="file://$(find lidarbot_description)/meshes/caster_mount.dae" /> -->
+          <mesh filename="package://lidarbot_description/meshes/caster_mount.dae" />
         </geometry>
       </visual>
@@ -51,6 +51,6 @@
         <origin xyz="-0.06 0.015 0.031" rpy="${pi} 0 ${-pi}"/>
           <geometry>
-              <mesh filename="file://$(find lidarbot_description)/meshes/rpi_stand.dae" />
-              <!-- <mesh filename="package://lidarbot_description/meshes/rpi_stand.dae" /> -->
+              <!-- <mesh filename="file://$(find lidarbot_description)/meshes/rpi_stand.dae" /> -->
+              <mesh filename="package://lidarbot_description/meshes/rpi_stand.dae" />
           </geometry>
       </visual>
@@ -65,6 +65,6 @@
         <origin xyz="-0.059 0.00245 0.033" rpy="0 0 ${pi/2}"/>
         <geometry>
-          <mesh filename="file://$(find lidarbot_description)/meshes/rpi_4.dae"/>
-          <!-- <mesh filename="package://lidarbot_description/meshes/rpi_4.dae"/> -->
+          <!-- <mesh filename="file://$(find lidarbot_description)/meshes/rpi_4.dae"/> -->
+          <mesh filename="package://lidarbot_description/meshes/rpi_4.dae"/>
         </geometry>
       </visual>
@@ -79,6 +79,6 @@
         <origin xyz="0.033 0.015 0.031" rpy="${pi} 0 ${pi}"/>
         <geometry>
-          <mesh filename="file://$(find lidarbot_description)/meshes/power_bank_stand.dae"/>
-          <!-- <mesh filename="package://lidarbot_description/meshes/power_bank_stand.dae"/> -->
+          <!-- <mesh filename="file://$(find lidarbot_description)/meshes/power_bank_stand.dae"/> -->
+          <mesh filename="package://lidarbot_description/meshes/power_bank_stand.dae"/>
         </geometry>
       </visual>
@@ -93,6 +93,6 @@
         <origin xyz="0.0635 0.04775 0.015" rpy="0 0 ${pi/2}"/>
         <geometry>
-          <mesh filename="file://$(find lidarbot_description)/meshes/power_bank.dae"/>
-          <!-- <mesh filename="package://lidarbot_description/meshes/power_bank.dae"/> -->
+          <!-- <mesh filename="file://$(find lidarbot_description)/meshes/power_bank.dae"/> -->
+          <mesh filename="package://lidarbot_description/meshes/power_bank.dae"/>
         </geometry>
       </visual>
@@ -107,6 +107,6 @@
         <origin xyz="0.033 0.015 0.017" rpy="0 0 ${-2*pi}"/>
         <geometry>
-          <mesh filename="file://$(find lidarbot_description)/meshes/rplidar_stand.dae"/>
-          <!-- <mesh filename="package://lidarbot_description/meshes/rplidar_stand.dae"/> -->
+          <!-- <mesh filename="file://$(find lidarbot_description)/meshes/rplidar_stand.dae"/> -->
+          <mesh filename="package://lidarbot_description/meshes/rplidar_stand.dae"/>
         </geometry>
       </visual>
@@ -121,6 +121,6 @@
         <origin xyz="0.03485 0.0087 0.037" rpy="0 0 ${-pi/2}"/>
           <geometry>
-            <mesh filename="file://$(find lidarbot_description)/meshes/rplidar_base.dae"/>
-            <!-- <mesh filename="package://lidarbot_description/meshes/rplidar_base.dae"/> -->
+            <!-- <mesh filename="file://$(find lidarbot_description)/meshes/rplidar_base.dae"/> -->
+            <mesh filename="package://lidarbot_description/meshes/rplidar_base.dae"/>
           </geometry>
         </visual>
@@ -152,6 +152,6 @@
     <visual>
         <geometry>
-          <mesh filename="file://$(find lidarbot_description)/meshes/left_wheel.dae" />
-          <!-- <mesh filename="package://lidarbot_description/meshes/left_wheel.dae" /> -->
+          <!-- <mesh filename="file://$(find lidarbot_description)/meshes/left_wheel.dae" /> -->
+          <mesh filename="package://lidarbot_description/meshes/left_wheel.dae" />
         </geometry>
     </visual>
@@ -176,6 +176,6 @@
     <visual>
       <geometry>
-        <mesh filename="file://$(find lidarbot_description)/meshes/right_wheel.dae"/>
-        <!-- <mesh filename="package://lidarbot_description/meshes/right_wheel.dae"/> -->
+        <!-- <mesh filename="file://$(find lidarbot_description)/meshes/right_wheel.dae"/> -->
+        <mesh filename="package://lidarbot_description/meshes/right_wheel.dae"/>
       </geometry>
     </visual>
@@ -200,6 +200,6 @@
     <visual>
       <geometry>
-        <mesh filename="file://$(find lidarbot_description)/meshes/caster_wheel.dae"/>
-        <!-- <mesh filename="package://lidarbot_description/meshes/caster_wheel.dae"/> -->
+        <!-- <mesh filename="file://$(find lidarbot_description)/meshes/caster_wheel.dae"/> -->
+        <mesh filename="package://lidarbot_description/meshes/caster_wheel.dae"/>
       </geometry>
     </visual>
