Commit message: Minor package changes

File: lidarbot_description/urdf/camera.xacro (robot description, xacro)
@@ -6,6 +6,6 @@
       <origin xyz="0 0 0" rpy="${pi/2} 0 ${pi/2}"/>
       <geometry>
-        <!-- <mesh filename="file://$(find lidarbot_description)/meshes/d415.dae"/> -->
-        <mesh filename="package://lidarbot_description/meshes/d415.dae"/>
+        <mesh filename="file://$(find lidarbot_description)/meshes/d415.dae"/>
+        <!-- <mesh filename="package://lidarbot_description/meshes/d415.dae"/> -->
       </geometry>
     </visual>

File: lidarbot_description/urdf/imu.xacro (robot description, xacro)
@@ -5,6 +5,6 @@
     <visual name="imu_visual">
       <geometry>
-        <!-- <mesh filename="file://$(find lidarbot_description)/meshes/MPU6050.dae"/> -->
-        <mesh filename="package://lidarbot_description/meshes/MPU6050.dae"/>
+        <mesh filename="file://$(find lidarbot_description)/meshes/MPU6050.dae"/>
+        <!-- <mesh filename="package://lidarbot_description/meshes/MPU6050.dae"/> -->
       </geometry>
     </visual>

File: lidarbot_description/urdf/lidar.xacro (robot description, xacro)
@@ -4,6 +4,6 @@
         <visual>
             <geometry>
-            <!-- <mesh filename="file://$(find lidarbot_description)/meshes/rplidar_top.dae"/> -->
-            <mesh filename="package://lidarbot_description/meshes/rplidar_top.dae"/>
+            <mesh filename="file://$(find lidarbot_description)/meshes/rplidar_top.dae"/>
+            <!-- <mesh filename="package://lidarbot_description/meshes/rplidar_top.dae"/> -->
             </geometry>
         </visual>

File: lidarbot_description/urdf/lidarbot_core.xacro (robot description, xacro)
@@ -24,6 +24,6 @@
         <origin xyz="0 0 ${-wheel_zoff}" rpy="0 0 0"/>
           <geometry>
-              <!-- <mesh filename="file://$(find lidarbot_description)/meshes/robot_chassis.dae" /> -->
-              <mesh filename="package://lidarbot_description/meshes/robot_chassis.dae" />
+              <mesh filename="file://$(find lidarbot_description)/meshes/robot_chassis.dae" />
+              <!-- <mesh filename="package://lidarbot_description/meshes/robot_chassis.dae" /> -->
           </geometry>
       </visual>
@@ -37,6 +37,6 @@
           <origin xyz="0.086 0 -0.0475" rpy="0 0 0"/>
         <geometry>
-          <!-- <mesh filename="file://$(find lidarbot_description)/meshes/caster_mount.dae" /> -->
-          <mesh filename="package://lidarbot_description/meshes/caster_mount.dae" />
+          <mesh filename="file://$(find lidarbot_description)/meshes/caster_mount.dae" />
+          <!-- <mesh filename="package://lidarbot_description/meshes/caster_mount.dae" /> -->
         </geometry>
       </visual>
@@ -51,6 +51,6 @@
         <origin xyz="-0.06 0.015 0.031" rpy="${pi} 0 ${-pi}"/>
           <geometry>
-              <!-- <mesh filename="file://$(find lidarbot_description)/meshes/rpi_stand.dae" /> -->
-              <mesh filename="package://lidarbot_description/meshes/rpi_stand.dae" />
+              <mesh filename="file://$(find lidarbot_description)/meshes/rpi_stand.dae" />
+              <!-- <mesh filename="package://lidarbot_description/meshes/rpi_stand.dae" /> -->
           </geometry>
       </visual>
@@ -65,6 +65,6 @@
         <origin xyz="-0.059 0.00245 0.033" rpy="0 0 ${pi/2}"/>
         <geometry>
-          <!-- <mesh filename="file://$(find lidarbot_description)/meshes/rpi_4.dae"/> -->
-          <mesh filename="package://lidarbot_description/meshes/rpi_4.dae"/>
+          <mesh filename="file://$(find lidarbot_description)/meshes/rpi_4.dae"/>
+          <!-- <mesh filename="package://lidarbot_description/meshes/rpi_4.dae"/> -->
         </geometry>
       </visual>
@@ -79,6 +79,6 @@
         <origin xyz="0.033 0.015 0.031" rpy="${pi} 0 ${pi}"/>
         <geometry>
-          <!-- <mesh filename="file://$(find lidarbot_description)/meshes/power_bank_stand.dae"/> -->
-          <mesh filename="package://lidarbot_description/meshes/power_bank_stand.dae"/>
+          <mesh filename="file://$(find lidarbot_description)/meshes/power_bank_stand.dae"/>
+          <!-- <mesh filename="package://lidarbot_description/meshes/power_bank_stand.dae"/> -->
         </geometry>
       </visual>
@@ -93,6 +93,6 @@
         <origin xyz="0.0635 0.04775 0.015" rpy="0 0 ${pi/2}"/>
         <geometry>
-          <!-- <mesh filename="file://$(find lidarbot_description)/meshes/power_bank.dae"/> -->
-          <mesh filename="package://lidarbot_description/meshes/power_bank.dae"/>
+          <mesh filename="file://$(find lidarbot_description)/meshes/power_bank.dae"/>
+          <!-- <mesh filename="package://lidarbot_description/meshes/power_bank.dae"/> -->
         </geometry>
       </visual>
@@ -107,6 +107,6 @@
         <origin xyz="0.033 0.015 0.017" rpy="0 0 ${-2*pi}"/>
         <geometry>
-          <!-- <mesh filename="file://$(find lidarbot_description)/meshes/rplidar_stand.dae"/> -->
-          <mesh filename="package://lidarbot_description/meshes/rplidar_stand.dae"/>
+          <mesh filename="file://$(find lidarbot_description)/meshes/rplidar_stand.dae"/>
+          <!-- <mesh filename="package://lidarbot_description/meshes/rplidar_stand.dae"/> -->
         </geometry>
       </visual>
@@ -121,6 +121,6 @@
         <origin xyz="0.03485 0.0087 0.037" rpy="0 0 ${-pi/2}"/>
           <geometry>
-            <!-- <mesh filename="file://$(find lidarbot_description)/meshes/rplidar_base.dae"/> -->
-            <mesh filename="package://lidarbot_description/meshes/rplidar_base.dae"/>
+            <mesh filename="file://$(find lidarbot_description)/meshes/rplidar_base.dae"/>
+            <!-- <mesh filename="package://lidarbot_description/meshes/rplidar_base.dae"/> -->
           </geometry>
         </visual>
@@ -152,6 +152,6 @@
     <visual>
         <geometry>
-          <!-- <mesh filename="file://$(find lidarbot_description)/meshes/left_wheel.dae" /> -->
-          <mesh filename="package://lidarbot_description/meshes/left_wheel.dae" />
+          <mesh filename="file://$(find lidarbot_description)/meshes/left_wheel.dae" />
+          <!-- <mesh filename="package://lidarbot_description/meshes/left_wheel.dae" /> -->
         </geometry>
     </visual>
@@ -176,6 +176,6 @@
     <visual>
       <geometry>
-        <!-- <mesh filename="file://$(find lidarbot_description)/meshes/right_wheel.dae"/> -->
-        <mesh filename="package://lidarbot_description/meshes/right_wheel.dae"/>
+        <mesh filename="file://$(find lidarbot_description)/meshes/right_wheel.dae"/>
+        <!-- <mesh filename="package://lidarbot_description/meshes/right_wheel.dae"/> -->
       </geometry>
     </visual>
@@ -200,6 +200,6 @@
     <visual>
       <geometry>
-        <!-- <mesh filename="file://$(find lidarbot_description)/meshes/caster_wheel.dae"/> -->
-        <mesh filename="package://lidarbot_description/meshes/caster_wheel.dae"/>
+        <mesh filename="file://$(find lidarbot_description)/meshes/caster_wheel.dae"/>
+        <!-- <mesh filename="package://lidarbot_description/meshes/caster_wheel.dae"/> -->
       </geometry>
     </visual>

Commit message: Update hardware interface to work with rviz

File: lidarbot_description/urdf/camera.xacro (robot description, xacro)
@@ -6,6 +6,5 @@
       <origin xyz="0 0 0" rpy="${pi/2} 0 ${pi/2}"/>
       <geometry>
-        <mesh filename="file://$(find lidarbot_description)/meshes/d415.dae"/>
-        <!-- <mesh filename="package://lidarbot_description/meshes/d415.dae"/> -->
+        <mesh filename="package://lidarbot_description/meshes/d415.dae"/>
       </geometry>
     </visual>

File: lidarbot_description/urdf/imu.xacro (robot description, xacro)
@@ -5,6 +5,5 @@
     <visual name="imu_visual">
       <geometry>
-        <mesh filename="file://$(find lidarbot_description)/meshes/MPU6050.dae"/>
-        <!-- <mesh filename="package://lidarbot_description/meshes/MPU6050.dae"/> -->
+        <mesh filename="package://lidarbot_description/meshes/MPU6050.dae"/>
       </geometry>
     </visual>

File: lidarbot_description/urdf/lidar.xacro (robot description, xacro)
@@ -4,6 +4,5 @@
         <visual>
             <geometry>
-            <mesh filename="file://$(find lidarbot_description)/meshes/rplidar_top.dae"/>
-            <!-- <mesh filename="package://lidarbot_description/meshes/rplidar_top.dae"/> -->
+                <mesh filename="package://lidarbot_description/meshes/rplidar_top.dae"/>
             </geometry>
         </visual>

File: lidarbot_description/urdf/lidarbot_core.xacro (robot description, xacro)
@@ -24,6 +24,5 @@
         <origin xyz="0 0 ${-wheel_zoff}" rpy="0 0 0"/>
           <geometry>
-              <mesh filename="file://$(find lidarbot_description)/meshes/robot_chassis.dae" />
-              <!-- <mesh filename="package://lidarbot_description/meshes/robot_chassis.dae" /> -->
+              <mesh filename="package://lidarbot_description/meshes/robot_chassis.dae" />
           </geometry>
       </visual>
@@ -37,6 +36,5 @@
           <origin xyz="0.086 0 -0.0475" rpy="0 0 0"/>
         <geometry>
-          <mesh filename="file://$(find lidarbot_description)/meshes/caster_mount.dae" />
-          <!-- <mesh filename="package://lidarbot_description/meshes/caster_mount.dae" /> -->
+          <mesh filename="package://lidarbot_description/meshes/caster_mount.dae" />
         </geometry>
       </visual>
@@ -51,6 +49,5 @@
         <origin xyz="-0.06 0.015 0.031" rpy="${pi} 0 ${-pi}"/>
           <geometry>
-              <mesh filename="file://$(find lidarbot_description)/meshes/rpi_stand.dae" />
-              <!-- <mesh filename="package://lidarbot_description/meshes/rpi_stand.dae" /> -->
+              <mesh filename="package://lidarbot_description/meshes/rpi_stand.dae" />
           </geometry>
       </visual>
@@ -65,6 +62,5 @@
         <origin xyz="-0.059 0.00245 0.033" rpy="0 0 ${pi/2}"/>
         <geometry>
-          <mesh filename="file://$(find lidarbot_description)/meshes/rpi_4.dae"/>
-          <!-- <mesh filename="package://lidarbot_description/meshes/rpi_4.dae"/> -->
+          <mesh filename="package://lidarbot_description/meshes/rpi_4.dae"/>
         </geometry>
       </visual>
@@ -79,6 +75,5 @@
         <origin xyz="0.033 0.015 0.031" rpy="${pi} 0 ${pi}"/>
         <geometry>
-          <mesh filename="file://$(find lidarbot_description)/meshes/power_bank_stand.dae"/>
-          <!-- <mesh filename="package://lidarbot_description/meshes/power_bank_stand.dae"/> -->
+          <mesh filename="package://lidarbot_description/meshes/power_bank_stand.dae"/>
         </geometry>
       </visual>
@@ -93,6 +88,5 @@
         <origin xyz="0.0635 0.04775 0.015" rpy="0 0 ${pi/2}"/>
         <geometry>
-          <mesh filename="file://$(find lidarbot_description)/meshes/power_bank.dae"/>
-          <!-- <mesh filename="package://lidarbot_description/meshes/power_bank.dae"/> -->
+          <mesh filename="package://lidarbot_description/meshes/power_bank.dae"/>
         </geometry>
       </visual>
@@ -107,6 +101,5 @@
         <origin xyz="0.033 0.015 0.017" rpy="0 0 ${-2*pi}"/>
         <geometry>
-          <mesh filename="file://$(find lidarbot_description)/meshes/rplidar_stand.dae"/>
-          <!-- <mesh filename="package://lidarbot_description/meshes/rplidar_stand.dae"/> -->
+          <mesh filename="package://lidarbot_description/meshes/rplidar_stand.dae"/>
         </geometry>
       </visual>
@@ -121,6 +114,5 @@
         <origin xyz="0.03485 0.0087 0.037" rpy="0 0 ${-pi/2}"/>
           <geometry>
-            <mesh filename="file://$(find lidarbot_description)/meshes/rplidar_base.dae"/>
-            <!-- <mesh filename="package://lidarbot_description/meshes/rplidar_base.dae"/> -->
+            <mesh filename="package://lidarbot_description/meshes/rplidar_base.dae"/>
           </geometry>
         </visual>
@@ -152,6 +144,5 @@
     <visual>
         <geometry>
-          <mesh filename="file://$(find lidarbot_description)/meshes/left_wheel.dae" />
-          <!-- <mesh filename="package://lidarbot_description/meshes/left_wheel.dae" /> -->
+          <mesh filename="package://lidarbot_description/meshes/left_wheel.dae" />
         </geometry>
     </visual>
@@ -176,6 +167,5 @@
     <visual>
       <geometry>
-        <mesh filename="file://$(find lidarbot_description)/meshes/right_wheel.dae"/>
-        <!-- <mesh filename="package://lidarbot_description/meshes/right_wheel.dae"/> -->
+        <mesh filename="package://lidarbot_description/meshes/right_wheel.dae"/>
       </geometry>
     </visual>
@@ -200,6 +190,5 @@
     <visual>
       <geometry>
-        <mesh filename="file://$(find lidarbot_description)/meshes/caster_wheel.dae"/>
-        <!-- <mesh filename="package://lidarbot_description/meshes/caster_wheel.dae"/> -->
+        <mesh filename="package://lidarbot_description/meshes/caster_wheel.dae"/>
       </geometry>
     </visual>

Commit message: Update some packages and README

File: lidarbot_description/urdf/camera.xacro (robot description, xacro)
@@ -6,5 +6,5 @@
       <origin xyz="0 0 0" rpy="${pi/2} 0 ${pi/2}"/>
       <geometry>
-        <mesh filename="package://lidarbot_description/meshes/d415.dae"/>
+        <mesh filename="package://lidarbot_description/meshes/rpi_camera.dae"/>
       </geometry>
     </visual>
@@ -33,5 +33,5 @@
         <update_rate>10</update_rate>
         <camera>
-            <horizontal_fov>1.089</horizontal_fov>
+            <horizontal_fov>0.934</horizontal_fov>
             <image>
                 <format>R8G8B8</format>

File: lidarbot_description/urdf/lidarbot_core.xacro (robot description, xacro)
@@ -129,9 +129,9 @@
         </geometry>
       </collision>
-      <!-- Depth camera mount -->
+      <!-- Camera mount -->
       <visual name="camera_mount_visual">
         <origin xyz="0.089 0 0.016" rpy="0 0 0"/>
           <geometry>
-            <cylinder radius="0.007" length="0.03"/>
+            <mesh filename="package://lidarbot_description/meshes/rpi_camera_mount.dae"/>
           </geometry>
       </visual>

File: lidarbot_description/urdf/ros2_control.xacro (robot description, xacro)
@@ -6,8 +6,8 @@
       <hardware>
         <plugin>lidarbot_base/LidarbotHardware</plugin>
-          <param name="left_wheel_name">left_wheel_joint</param>
-          <param name="right_wheel_name">right_wheel_joint</param>
-          <param name="enc_ticks_per_rev">20</param>
-          <param name="loop_rate">30.0</param>
+          <param name='left_wheel_name'>left_wheel_joint</param>
+          <param name='right_wheel_name'>right_wheel_joint</param>
+          <param name='enc_ticks_per_rev'>20</param>
+          <param name='loop_rate'>30.0</param>
       </hardware>
       <joint name='left_wheel_joint'>
@@ -28,4 +28,19 @@
       </joint>
     </ros2_control>
+	<!-- Imu sensor broadcaster -->
+	<ros2_control name='IMUSensorBroadcaster' type='sensor'>
+	  <hardware>
+		<plugin>imu_sensor_broadcaster/IMUSensorBroadcaster</plugin>
+	  </hardware>
+	  <sensor name='mpu6050'>
+		<param name='frame_id'>imu_link</param>
+		<state_interface name='angular_velocity.x'/>
+		<state_interface name='angular_velocity.y'/>
+		<state_interface name='angular_velocity.z'/>
+		<state_interface name='linear_acceleration.x'/>
+		<state_interface name='linear_acceleration.y'/>
+		<state_interface name='linear_acceleration.z'/>
+	  </sensor>
+	</ros2_control>
   </xacro:unless>
   <!-- Gazebo ros2_control -->

Commit message: Update URDF and mesh files

File: lidarbot_description/urdf/camera.xacro (robot description, xacro)
@@ -4,15 +4,9 @@
   <link name="camera_link">
     <visual>
-      <origin xyz="0 0 0" rpy="${pi/2} 0 ${pi/2}"/>
+      <origin xyz="-0.0115 0.0125 0.0052" rpy="1.8745 ${pi} ${pi/2}"/>
       <geometry>
         <mesh filename="package://lidarbot_description/meshes/rpi_camera.dae"/>
       </geometry>
     </visual>
-    <collision>
-      <origin xyz="-0.012 0 0" rpy="0 0 ${pi/2}"/>
-      <geometry>
-        <box size="0.1 0.025 0.022"/>
-      </geometry>
-    </collision>
   </link>
   <joint name="camera_joint" type="fixed">
@@ -30,5 +24,5 @@
     <sensor name="camera" type="camera">
         <pose> 0 0 0 0 0 0 </pose>
-        <visualize>true</visualize>
+        <visualize>false</visualize>
         <update_rate>10</update_rate>
         <camera>

File: lidarbot_description/urdf/lidarbot_core.xacro (robot description, xacro)
@@ -131,5 +131,5 @@
       <!-- Camera mount -->
       <visual name="camera_mount_visual">
-        <origin xyz="0.089 0 0.016" rpy="0 0 0"/>
+        <origin xyz="0.055 0.0335 0.001" rpy="0 0 ${pi}"/>
           <geometry>
             <mesh filename="package://lidarbot_description/meshes/rpi_camera_mount.dae"/>
@@ -137,7 +137,7 @@
       </visual>
       <collision name="camera_mount_collision">
-        <origin xyz="0.089 0 0.016" rpy="0 0 0"/>
-        <geometry>
-          <cylinder radius="0.008" length="0.031"/>
+        <origin xyz="0.075 0.0335 0.015" rpy="0 ${-pi/2} 0"/>
+        <geometry>
+          <box size="0.035 0.06 0.02"/>
         </geometry>
       </collision>

File: lidarbot_description/urdf/ros2_control.xacro (robot description, xacro)
@@ -29,5 +29,5 @@
     </ros2_control>
 	<!-- Imu sensor broadcaster -->
-	<ros2_control name='IMUSensorBroadcaster' type='sensor'>
+	<!--<ros2_control name='IMUSensorBroadcaster' type='sensor'>
 	  <hardware>
 		<plugin>imu_sensor_broadcaster/IMUSensorBroadcaster</plugin>
@@ -42,5 +42,5 @@
 		<state_interface name='linear_acceleration.z'/>
 	  </sensor>
-	</ros2_control>
+	</ros2_control> -->
   </xacro:unless>
   <!-- Gazebo ros2_control -->
