Commit message: Update xacro files, slam and teleop packages
Signed-off-by: TheNoobInventor <eduobijoro@mailfence.com>

File: lidarbot_description/urdf/camera.xacro (robot description, xacro)
@@ -13,5 +13,5 @@
     <parent link="chassis_link"/>
     <child link="camera_link"/>
-    <origin xyz="0.1 0 0.0425" rpy="0 0 0"/>
+    <origin xyz="0.205 0 0.0425" rpy="0 0 0"/>
   </joint>
   <link name="camera_link_optical"></link>

File: lidarbot_description/urdf/imu.xacro (robot description, xacro)
@@ -12,5 +12,5 @@
     <parent link="chassis_link"/>
     <child link="imu_link"/>
-    <origin xyz="-0.06 0 0.0175" rpy="0 0 ${pi}"/>
+    <origin xyz="0.045 0 0.0175" rpy="0 0 ${pi}"/>
   </joint>
 </robot>

File: lidarbot_description/urdf/lidar.xacro (robot description, xacro)
@@ -3,4 +3,5 @@
     <link name="lidar_link">
         <visual>
+            <origin xyz="0 -0.0009 -0.011" rpy="0 0 0"/>
             <geometry>
                 <mesh filename="package://lidarbot_description/meshes/rplidar_top.dae"/>
@@ -8,10 +9,10 @@
         </visual>
         <collision>
-            <origin xyz="0 -0.0009 0.011" rpy="0 0 0"/>
+            <origin xyz="0 -0.0028 0" rpy="0 0 0"/>
             <geometry>
-            <cylinder radius="0.037" length="0.021"/>
+                <cylinder radius="0.037" length="0.021"/>
             </geometry>
         </collision>
-         <xacro:cylinder_inertia mass="${wheel_mass}" length="0.021" radius="0.037">
+         <xacro:cylinder_inertia mass="0.07" length="0.021" radius="0.037">
             <origin xyz="0 0 0" rpy="0 0 0"/>
         </xacro:cylinder_inertia>
@@ -20,11 +21,12 @@
         <parent link="chassis_link"/>
         <child link="lidar_link"/>
-        <origin xyz="0.0335 0.0095 0.069" rpy="0 0 ${-pi/2}"/>
+        <origin xyz="0.1385 0.0095 0.08" rpy="0 0 ${-pi/2}"/>
         <axis xyz="0 0 1"/>
     </joint>
     <gazebo reference="lidar_link">
         <sensor name="lidar" type="ray">
-            <pose> 0 0 0 0 0 0 </pose>
-            <visualize>false</visualize>
+            <pose>0 0 0 0 0 0</pose>
+            <always_on>true</always_on>
+            <visualize>true</visualize>
             <update_rate>10</update_rate>
             <ray>
@@ -37,7 +39,14 @@
                 </scan>
                 <range>
-                    <min>0.3</min>
-                    <max>12</max>
-                </range>
+                    <min>0.15</min>
+                    <max>6.0</max>
+                    <!-- <max>12.0</max> -->
+                    <resolution>0.01500</resolution>
+		        </range>
+                <noise>
+                    <type>gaussian</type>
+                    <mean>0.0</mean>
+                    <stddev>0.01</stddev>
+                </noise>
             </ray>
             <plugin name="lidar_controller" filename="libgazebo_ros_ray_sensor.so">

File: lidarbot_description/urdf/lidarbot_core.xacro (robot description, xacro)
@@ -17,5 +17,5 @@
      <parent link="base_link"/>
      <child link="chassis_link"/>
-     <origin xyz="0 0 -${(wheel_radius+wheel_zoff)}" rpy="0 0 0"/>
+     <origin xyz="-0.076 0 0" rpy="0 0 0"/>
    </joint>
   <link name="base_footprint"/>
@@ -23,10 +23,10 @@
     <parent link="base_link"/>
     <child link="base_footprint"/>
-    <origin xyz="0 0 -${2*(wheel_radius)+wheel_zoff}" rpy="0 0 0"/>
+    <origin xyz="0 0 -${(wheel_radius + wheel_zoff / 2)}" rpy="0 0 0"/>
   </joint>
   <!-- Robot Chassis -->
   <link name="chassis_link">
       <visual>
-        <origin xyz="0 0 ${-wheel_zoff}" rpy="0 0 0"/>
+        <origin xyz="${base_length/2} 0 ${-wheel_zoff}" rpy="0 0 0"/>
           <geometry>
               <mesh filename="package://lidarbot_description/meshes/robot_chassis.dae" />
@@ -34,4 +34,5 @@
       </visual>
       <collision>
+        <origin xyz="${base_length/2} 0 ${-wheel_zoff}" rpy="0 0 0"/>
         <geometry>
           <box size="${base_length} ${base_width} ${base_height}"/>
@@ -40,5 +41,5 @@
     <!-- Caster mount -->
       <visual name="caster_mount_visual">
-          <origin xyz="0.086 0 -0.0475" rpy="0 0 0"/>
+          <origin xyz="0.191 0 -0.0475" rpy="0 0 0"/>
         <geometry>
           <mesh filename="package://lidarbot_description/meshes/caster_mount.dae" />
@@ -46,5 +47,5 @@
       </visual>
       <collision name="caster_mount_collision">
-        <origin xyz="0.086 0 -0.005" rpy="0 0 0"/>
+        <origin xyz="0.191 0 -0.005" rpy="0 0 0"/>
         <geometry>
           <cylinder radius="0.023" length="0.0125"/>
@@ -53,5 +54,5 @@
       <!-- Rpi stand -->
       <visual name="rpi_4_stand_visual">
-        <origin xyz="-0.06 0.015 0.031" rpy="${pi} 0 ${-pi}"/>
+        <origin xyz="0.045 0.015 0.031" rpy="${pi} 0 ${-pi}"/>
           <geometry>
               <mesh filename="package://lidarbot_description/meshes/rpi_stand.dae" />
@@ -59,5 +60,5 @@
       </visual>
       <collision name="rpi_4_stand_collision">
-        <origin xyz="-0.06 0 0.017" rpy="0 0 ${pi/2}"/>
+        <origin xyz="0.045 0 0.017" rpy="0 0 ${pi/2}"/>
         <geometry>
           <box size="0.098 0.065 0.034"/>
@@ -66,5 +67,5 @@
       <!-- Raspberry Pi -->
       <visual name="rpi_4_visual">
-        <origin xyz="-0.059 0.00245 0.033" rpy="0 0 ${pi/2}"/>
+        <origin xyz="0.046 0.00245 0.033" rpy="0 0 ${pi/2}"/>
         <geometry>
           <mesh filename="package://lidarbot_description/meshes/rpi_4.dae"/>
@@ -72,5 +73,5 @@
       </visual>
       <collision name="rpi_4_collision">
-        <origin xyz="-0.058 0.005 0.041" rpy="0 0 ${pi/2}"/>
+        <origin xyz="0.047 0.005 0.041" rpy="0 0 ${pi/2}"/>
         <geometry>
           <box size="0.09 0.06 0.02"/>
@@ -79,5 +80,5 @@
       <!-- Power bank stand -->
       <visual name="power_bank_stand_visual">
-        <origin xyz="0.033 0.015 0.031" rpy="${pi} 0 ${pi}"/>
+        <origin xyz="0.138 0.015 0.031" rpy="${pi} 0 ${pi}"/>
         <geometry>
           <mesh filename="package://lidarbot_description/meshes/power_bank_stand.dae"/>
@@ -85,5 +86,5 @@
       </visual>
       <collision name="power_bank_stand_collision">
-        <origin xyz="0.033 0 0.0085" rpy="0 0 ${pi/2}"/>
+        <origin xyz="0.138 0 0.0085" rpy="0 0 ${pi/2}"/>
         <geometry>
           <box size="0.098 0.065 0.015"/>
@@ -92,5 +93,5 @@
       <!-- Power bank -->
       <visual name="power_bank_visual">
-        <origin xyz="0.0635 0.04775 0.015" rpy="0 0 ${pi/2}"/>
+        <origin xyz="0.1685 0.04775 0.015" rpy="0 0 ${pi/2}"/>
         <geometry>
           <mesh filename="package://lidarbot_description/meshes/power_bank.dae"/>
@@ -98,5 +99,5 @@
       </visual>
       <collision name="power_bank_collision">
-        <origin xyz="0.033 0 0.025" rpy="0 0 ${pi/2}"/>
+        <origin xyz="0.138 0 0.025" rpy="0 0 ${pi/2}"/>
         <geometry>
           <box size="0.096 0.062 0.02"/>
@@ -105,5 +106,5 @@
       <!-- Rplidar stand -->
       <visual name="rplidar_stand_visual">
-        <origin xyz="0.033 0.015 0.017" rpy="0 0 ${-2*pi}"/>
+        <origin xyz="0.138 0.015 0.017" rpy="0 0 ${-2*pi}"/>
         <geometry>
           <mesh filename="package://lidarbot_description/meshes/rplidar_stand.dae"/>
@@ -111,5 +112,5 @@
       </visual>
       <collision name="rplidar_stand_collision">
-        <origin xyz="0.033 0 0.04" rpy="0 0 ${pi/2}"/>
+        <origin xyz="0.138 0 0.04" rpy="0 0 ${pi/2}"/>
         <geometry>
           <box size="0.098 0.065 0.015"/>
@@ -118,5 +119,5 @@
       <!-- Rplidar base -->
       <visual name="rplidar_base_visual">
-        <origin xyz="0.03485 0.0087 0.037" rpy="0 0 ${-pi/2}"/>
+        <origin xyz="0.13985 0.0087 0.037" rpy="0 0 ${-pi/2}"/>
           <geometry>
             <mesh filename="package://lidarbot_description/meshes/rplidar_base.dae"/>
@@ -124,12 +125,12 @@
         </visual>
       <collision name="rplidar_base_collision">
-        <origin xyz="0.033 0 0.056" rpy="0 0 ${-pi/2}"/>
-        <geometry>
-          <box size="0.12 0.072 0.035"/>
+        <origin xyz="0.138 0 0.056" rpy="0 0 ${-pi/2}"/>
+        <geometry>
+          <box size="0.11 0.072 0.035"/>
         </geometry>
       </collision>
       <!-- Camera mount -->
       <visual name="camera_mount_visual">
-        <origin xyz="0.055 0.0335 0.001" rpy="0 0 ${pi}"/>
+        <origin xyz="0.16 0.0335 0.001" rpy="0 0 ${pi}"/>
           <geometry>
             <mesh filename="package://lidarbot_description/meshes/rpi_camera_mount.dae"/>
@@ -137,11 +138,11 @@
       </visual>
       <collision name="camera_mount_collision">
-        <origin xyz="0.092 0.0 0.035" rpy="${pi/2} 0 ${pi/2}"/>
-        <geometry>
-          <box size="0.045 0.04 0.02"/>
+        <origin xyz="0.197 0.0 0.032" rpy="${pi/2} 0 ${pi/2}"/>
+        <geometry>
+          <box size="0.048 0.06 0.033"/>
         </geometry>
       </collision>
     <xacro:box_inertia mass="0.864" length="${base_length}" width="${base_width}" height="${base_height}">
-      <origin xyz="0 0 -0.0125" rpy="0 0 0"/>
+      <origin xyz="0.105 0 0.0175" rpy="0 0 0"/>
     </xacro:box_inertia>
   </link>
@@ -166,5 +167,5 @@
     <parent link="chassis_link"/>
     <child link="left_wheel"/>
-    <origin xyz="-0.028 0.055 -${wheel_zoff}" rpy="${pi/2} 0 ${pi}"/>
+    <origin xyz="0.077 0.055 -${wheel_zoff}" rpy="${pi/2} 0 ${pi}"/>
     <axis xyz="0 0 1"/>
   </joint>
@@ -189,5 +190,5 @@
     <parent link="chassis_link"/>
     <child link="right_wheel"/>
-    <origin xyz="-0.028 -0.065 -${wheel_zoff}" rpy="${pi/2} 0 ${-pi}"/>
+    <origin xyz="0.077 -0.065 -${wheel_zoff}" rpy="${pi/2} 0 ${-pi}"/>
     <axis xyz="0 0 1"/>
   </joint>
@@ -212,5 +213,5 @@
     <parent link="chassis_link"/>
     <child link="caster_wheel"/>
-    <origin xyz="0.0925 0 -0.031" rpy="0 0 ${pi/2}"/>
+    <origin xyz="0.1975 0 -0.031" rpy="0 0 ${pi/2}"/>
   </joint>
   <gazebo reference="caster_wheel">

Commit message: Update package.xml files and README

File: lidarbot_description/urdf/camera.xacro (robot description, xacro)
@@ -11,5 +11,5 @@
   </link>
   <joint name="camera_joint" type="fixed">
-    <parent link="chassis_link"/>
+    <parent link="base_link"/>
     <child link="camera_link"/>
     <origin xyz="0.205 0 0.0425" rpy="0 0 0"/>

File: lidarbot_description/urdf/gazebo_control.xacro (robot description, xacro)
@@ -13,5 +13,5 @@
             <!-- Output -->
             <odometry_frame>odom</odometry_frame>
-            <robot_base_frame>base_link</robot_base_frame>
+            <robot_base_frame>base_footprint</robot_base_frame>
             <publish_odom>true</publish_odom>
             <publish_odom_tf>true</publish_odom_tf>

File: lidarbot_description/urdf/imu.xacro (robot description, xacro)
@@ -10,8 +10,7 @@
   </link>
   <joint name="imu_joint" type="fixed">
-    <parent link="chassis_link"/>
+    <parent link="base_link"/>
     <child link="imu_link"/>
     <origin xyz="0.045 0 0.0175" rpy="0 0 0"/>
-    <!-- <origin xyz="0.045 0 0.0175" rpy="0 0 ${pi}"/> -->
   </joint>
  <gazebo reference="imu_link">

File: lidarbot_description/urdf/lidar.xacro (robot description, xacro)
@@ -19,5 +19,5 @@
    </link>
     <joint name="lidar_joint" type="fixed">
-        <parent link="chassis_link"/>
+        <parent link="base_link"/>
         <child link="lidar_link"/>
         <origin xyz="0.1385 0.0095 0.08" rpy="0 0 ${-pi/2}"/>

File: lidarbot_description/urdf/lidarbot_core.xacro (robot description, xacro)
@@ -2,5 +2,5 @@
 <robot xmlns:xacro="http://ros.org/wiki/xacro">
   <xacro:include filename="inertial_macros.xacro"/>
-  <!-- Robot's chassis properties -->
+  <!-- Robot's base properties -->
   <xacro:property name="base_length" value="0.21"/>
   <xacro:property name="base_width" value="0.11"/>
@@ -10,21 +10,22 @@
   <xacro:property name="wheel_height" value="0.025"/>
   <xacro:property name="wheel_mass" value="0.031"/>
-  <!-- Distance between centre of wheel and robot base/chassis -->
+  <!-- Distance between centre of wheel and robot base/base -->
   <xacro:property name="wheel_zoff" value="0.0125"/>
-   <!-- Base link -->
-   <link name="base_link"/>
-   <joint name="chassis_joint" type="fixed">
-     <parent link="base_link"/>
-     <child link="chassis_link"/>
-     <origin xyz="-0.076 0 0" rpy="0 0 0"/>
+  <link name="base_footprint"/>
+   <joint name="base_joint" type="fixed">
+     <parent link="base_footprint"/>
+     <child link="base_link"/>
+     <!-- <origin xyz="-0.076 0 0" rpy="0 0 0"/> -->
+     <origin xyz="-0.076 0 ${(wheel_radius + wheel_zoff / 2)}" rpy="0 0 0"/>
    </joint>
-  <link name="base_footprint"/>
-  <joint name="base_footprint_joint" type="fixed">
-    <parent link="base_link"/>
-    <child link="base_footprint"/>
-    <origin xyz="0 0 -${(wheel_radius + wheel_zoff / 2)}" rpy="0 0 0"/>
-  </joint>
-  <!-- Robot Chassis -->
-  <link name="chassis_link">
+  <!-- <joint name="base_footprint_joint" type="fixed">
+    <parent link="base_footprint"/>
+    <child link="base_link"/> -->
+    <!-- <parent link="base_link"/> -->
+    <!-- <child link="base_footprint"/> -->
+    <!-- <origin xyz="0 0 -${(wheel_radius + wheel_zoff / 2)}" rpy="0 0 0"/>
+  </joint> -->
+  <!-- Robot base chasis-->
+  <link name="base_link">
       <visual>
         <origin xyz="${base_length/2} 0 ${-wheel_zoff}" rpy="0 0 0"/>
@@ -165,5 +166,5 @@
   </link>
   <joint name="left_wheel_joint" type="continuous">
-    <parent link="chassis_link"/>
+    <parent link="base_link"/>
     <child link="left_wheel"/>
     <origin xyz="0.077 0.055 -${wheel_zoff}" rpy="${pi/2} 0 ${pi}"/>
@@ -188,5 +189,5 @@
   </link>
   <joint name="right_wheel_joint" type="continuous">
-    <parent link="chassis_link"/>
+    <parent link="base_link"/>
     <child link="right_wheel"/>
     <origin xyz="0.077 -0.065 -${wheel_zoff}" rpy="${pi/2} 0 ${-pi}"/>
@@ -211,5 +212,5 @@
   </link>
   <joint name="caster_wheel_joint" type="fixed">
-    <parent link="chassis_link"/>
+    <parent link="base_link"/>
     <child link="caster_wheel"/>
     <origin xyz="0.1975 0 -0.031" rpy="0 0 ${pi/2}"/>
