Commit message: Include program to generate imu covariances

File: lidarbot_description/urdf/imu.xacro (robot description, xacro)
@@ -12,5 +12,6 @@
     <parent link="chassis_link"/>
     <child link="imu_link"/>
-    <origin xyz="0.045 0 0.0175" rpy="0 0 ${pi}"/>
+    <origin xyz="0.045 0 0.0175" rpy="0 0 0"/>
+    <!-- <origin xyz="0.045 0 0.0175" rpy="0 0 ${pi}"/> -->
   </joint>
  <gazebo reference="imu_link">

Commit message: Minor update to some xacro files and README

File: lidarbot_description/urdf/imu.xacro (robot description, xacro)
@@ -18,5 +18,5 @@
     <plugin name="imu_controller" filename="libgazebo_ros_imu_sensor.so">
        <ros>
-         <remapping>~/out:=imu_broadcaster/imu</remapping>
+         <remapping>~/out:=imu_broadcaster/data</remapping>
        </ros>
       <initial_orientation_as_reference>false</initial_orientation_as_reference>

File: lidarbot_description/urdf/lidarbot_core.xacro (robot description, xacro)
@@ -16,14 +16,6 @@
      <parent link="base_footprint"/>
      <child link="base_link"/>
-     <!-- <origin xyz="-0.076 0 0" rpy="0 0 0"/> -->
      <origin xyz="-0.076 0 ${(wheel_radius + wheel_zoff / 2)}" rpy="0 0 0"/>
    </joint>
-  <!-- <joint name="base_footprint_joint" type="fixed">
-    <parent link="base_footprint"/>
-    <child link="base_link"/> -->
-    <!-- <parent link="base_link"/> -->
-    <!-- <child link="base_footprint"/> -->
-    <!-- <origin xyz="0 0 -${(wheel_radius + wheel_zoff / 2)}" rpy="0 0 0"/>
-  </joint> -->
   <!-- Robot base chasis-->
   <link name="base_link">

File: lidarbot_description/urdf/ros2_control.xacro (robot description, xacro)
@@ -27,6 +27,6 @@
         <state_interface name='position'/>
       </joint>
-	  </ros2_control>
-	  <!-- MPU6050 sensor-->
+    </ros2_control>
+    <!-- MPU6050 sensor-->
     <ros2_control name='MPU6050' type='sensor'>
       <hardware>
