Commit message: Minor edit to lidarbot_core.xacro

File: lidarbot_description/urdf/lidarbot_core.xacro (robot description, xacro)
@@ -19,4 +19,11 @@
      <origin xyz="0 0 -${(wheel_radius+wheel_zoff)}" rpy="0 0 0"/>
    </joint>
+  <link name="base_footprint"/>
+  <joint name="base_footprint_joint" type="fixed">
+    <parent link="base_link"/>
+    <child link="base_footprint"/>
+    <origin xyz="0 0 -${(wheel_radius+wheel_zoff)" rpy="0 0 0"/>
+	  <!-- <origin xyz="0 0 0" rpy="0 0 0"/> -->
+  </joint>
   <!-- Robot Chassis -->
   <link name="chassis_link">

Commit message: Add config file for lidarbot_slam

File: lidarbot_description/urdf/lidarbot_core.xacro (robot description, xacro)
@@ -23,5 +23,5 @@
     <parent link="base_link"/>
     <child link="base_footprint"/>
-    <origin xyz="0 0 -${(wheel_radius+wheel_zoff)" rpy="0 0 0"/>
+    <origin xyz="0 0 ${(wheel_radius+wheel_zoff)" rpy="0 0 0"/>
 	  <!-- <origin xyz="0 0 0" rpy="0 0 0"/> -->
   </joint>

Commit message: Update description and gazebo packages

File: lidarbot_description/urdf/lidarbot_core.xacro (robot description, xacro)
@@ -23,6 +23,5 @@
     <parent link="base_link"/>
     <child link="base_footprint"/>
-    <origin xyz="0 0 ${(wheel_radius+wheel_zoff)" rpy="0 0 0"/>
-	  <!-- <origin xyz="0 0 0" rpy="0 0 0"/> -->
+    <origin xyz="0 0 -${2*(wheel_radius)+wheel_zoff}" rpy="0 0 0"/>
   </joint>
   <!-- Robot Chassis -->

Commit message: Update README, teleop config and launch files

File: lidarbot_description/urdf/lidarbot_core.xacro (robot description, xacro)
@@ -137,7 +137,7 @@
       </visual>
       <collision name="camera_mount_collision">
-        <origin xyz="0.075 0.0335 0.015" rpy="0 ${-pi/2} 0"/>
-        <geometry>
-          <box size="0.035 0.06 0.02"/>
+        <origin xyz="0.092 0.0 0.035" rpy="${pi/2} 0 ${pi/2}"/>
+        <geometry>
+          <box size="0.045 0.04 0.02"/>
         </geometry>
       </collision>

Commit message: Update README and images after changing wheel positions

File: lidarbot_description/urdf/lidarbot_core.xacro (robot description, xacro)
@@ -21,5 +21,5 @@
   <link name="base_link">
       <visual>
-        <origin xyz="${base_length/2} 0 ${-wheel_zoff}" rpy="0 0 0"/>
+        <origin xyz="${base_length/2} 0 ${-wheel_zoff}" rpy="0 0 ${pi}"/>
           <geometry>
               <mesh filename="package://lidarbot_description/meshes/robot_chassis.dae" />
@@ -34,5 +34,5 @@
     <!-- Caster mount -->
       <visual name="caster_mount_visual">
-          <origin xyz="0.191 0 -0.0475" rpy="0 0 0"/>
+          <origin xyz="0.0185 0 -0.0475" rpy="0 0 0"/>
         <geometry>
           <mesh filename="package://lidarbot_description/meshes/caster_mount.dae" />
@@ -40,5 +40,5 @@
       </visual>
       <collision name="caster_mount_collision">
-        <origin xyz="0.191 0 -0.005" rpy="0 0 0"/>
+        <origin xyz="0.0185 0 -0.005" rpy="0 0 0"/>
         <geometry>
           <cylinder radius="0.023" length="0.0125"/>
@@ -160,5 +160,5 @@
     <parent link="base_link"/>
     <child link="left_wheel"/>
-    <origin xyz="0.077 0.055 -${wheel_zoff}" rpy="${pi/2} 0 ${pi}"/>
+    <origin xyz="0.133 0.055 -${wheel_zoff}" rpy="${pi/2} 0 ${pi}"/>
     <axis xyz="0 0 1"/>
   </joint>
@@ -183,5 +183,5 @@
     <parent link="base_link"/>
     <child link="right_wheel"/>
-    <origin xyz="0.077 -0.065 -${wheel_zoff}" rpy="${pi/2} 0 ${-pi}"/>
+    <origin xyz="0.133 -0.065 -${wheel_zoff}" rpy="${pi/2} 0 ${-pi}"/>
     <axis xyz="0 0 1"/>
   </joint>
@@ -206,5 +206,5 @@
     <parent link="base_link"/>
     <child link="caster_wheel"/>
-    <origin xyz="0.1975 0 -0.031" rpy="0 0 ${pi/2}"/>
+    <origin xyz="0.028 0 -0.031" rpy="0 0 ${pi/2}"/>
   </joint>
   <gazebo reference="caster_wheel">

Commit message: Minor update to wheel joints lidarbot_core.xacro

File: lidarbot_description/urdf/lidarbot_core.xacro (robot description, xacro)
@@ -144,5 +144,5 @@
     <visual>
         <geometry>
-          <mesh filename="package://lidarbot_description/meshes/left_wheel.dae" />
+          <mesh filename="package://lidarbot_description/meshes/right_wheel.dae" />
         </geometry>
     </visual>
@@ -160,5 +160,5 @@
     <parent link="base_link"/>
     <child link="left_wheel"/>
-    <origin xyz="0.133 0.055 -${wheel_zoff}" rpy="${pi/2} 0 ${pi}"/>
+    <origin xyz="0.133 0.065 -${wheel_zoff}" rpy="-${pi/2} 0 ${pi}"/>
     <axis xyz="0 0 1"/>
   </joint>

Commit message: Update trajectory_visualizer node

File: lidarbot_description/urdf/lidarbot_core.xacro (robot description, xacro)
@@ -140,5 +140,5 @@
     </xacro:box_inertia>
   </link>
-  <!-- Left Wheel -->
+  <!-- Left wheel -->
   <link name="left_wheel">
     <visual>
@@ -148,5 +148,5 @@
     </visual>
     <collision>
-      <origin xyz="0 0 0.0155" rpy="0 0 0"/>
+      <origin xyz="0 0 -0.0065" rpy="0 0 0"/>
       <geometry>
         <sphere radius="${wheel_radius}"/>
@@ -161,7 +161,7 @@
     <child link="left_wheel"/>
     <origin xyz="0.133 0.065 -${wheel_zoff}" rpy="-${pi/2} 0 ${pi}"/>
-    <axis xyz="0 0 1"/>
+    <axis xyz="0 0 -1"/>
   </joint>
-  <!-- Right Wheel -->
+  <!-- Right wheel -->
   <link name="right_wheel">
     <visual>
@@ -212,3 +212,11 @@
     <mu2 value="0.001"/>
   </gazebo>
+  <gazebo reference="left_wheel">
+    <mu1 value="1.16"/>
+    <mu2 value="1.16"/>
+  </gazebo>
+  <gazebo reference="right_wheel">
+    <mu1 value="1.16"/>
+    <mu2 value="1.16"/>
+  </gazebo>
 </robot>
